File: HW/rpi_pico_media_board/rpi_pico_media_board.kicad_sch (KiCad schematic)
At the start: 0 parts

Commit message: Scheme improvements
Changed lines of the file:
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@@
 	)
 	(sheet
-		(at 241.3 50.8)
+		(at 127 101.6)
 		(size 25.4 25.4)
 		(fields_autoplaced yes)
@@
 		)
 		(property "Sheetname" "[6]I2C_Peripherals"
-			(at 241.3 50.0884 0)
+			(at 127 100.8884 0)
 			(effects
 				(font
@@
 		)
 		(property "Sheetfile" "[6]I2C_Peripherals.kicad_sch"
-			(at 241.3 76.7846 0)
+			(at 127 127.5846 0)
 			(effects
 				(font
@@
 	)
 	(sheet
-		(at 165.1 50.8)
+		(at 50.8 101.6)
 		(size 25.4 25.4)
 		(fields_autoplaced yes)
@@
 		)
 		(property "Sheetname" "[4]TF_CARD"
-			(at 165.1 50.0884 0)
+			(at 50.8 100.8884 0)
 			(effects
 				(font
@@
 		)
 		(property "Sheetfile" "[4]TF_CARD.kicad_sch"
-			(at 165.1 76.7846 0)
+			(at 50.8 127.5846 0)
 			(effects
 				(font
@@
 	)
 	(sheet
-		(at 203.2 50.8)
+		(at 88.9 101.6)
 		(size 25.4 25.4)
 		(fields_autoplaced yes)
@@
 		)
 		(property "Sheetname" "[5]Macro_Pad"
-			(at 203.2 50.0884 0)
+			(at 88.9 100.8884 0)
 			(effects
 				(font
@@
 		)
 		(property "Sheetfile" "[5]Macro_Pad.kicad_sch"
-			(at 203.2 76.7846 0)
+			(at 88.9 127.5846 0)
 			(effects
 				(font
