File: HW/rpi_pico_media_board/[6]I2C_Peripherals.kicad_sch (KiCad schematic)
At the start: 11 parts, among them U5 PCF8563TS, Y1 32768Hz

Commit message: Scheme improvements
Parts:
- renumbered BT1 to BT600, Brd1 to Brd600, C27 to C600, C28 to C601, C26 to C602, D10 to D600, D11 to D601, R24 to R600, R25 to R601, U5 to U600, Y1 to Y600
Connections:
- net I2C_SCL renamed I2C1_SCL
- net I2C_SDA renamed I2C1_SDA
Other:
- note added: "SSD1306 LCD"
- note added: "[6]I2C Peripherals"
- note removed: "LCD"
Changed lines of the file:
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@@
 		)
 	)
-	(text "LCD"
-		(exclude_from_sim no)
-		(at 184.912 30.988 0)
+	(text "[6]I2C Peripherals"
+		(exclude_from_sim no)
+		(at 43.18 19.812 0)
 		(effects
 			(font
-				(size 1.27 1.27)
-			)
-		)
-	)
-	(text "RTC module\nPCF8563"
-		(exclude_from_sim no)
-		(at 26.67 35.052 0)
+				(size 3.81 3.81)
+			)
+		)
+	)
+	(text "SSD1306 LCD"
+		(exclude_from_sim no)
+		(at 196.088 29.972 0)
 		(effects
 			(font
-				(size 1.27 1.27)
+				(size 2.54 2.54)
+			)
+		)
+	)
+	(text "RTC module PCF8563"
+		(exclude_from_sim no)
+		(at 39.878 28.194 0)
+		(effects
+			(font
+				(size 2.54 2.54)
 			)
 		)
@@
 			)
 			(justify left bottom)
-		)
-	)
-	(global_label "I2C_SDA"
-		(shape input)
-		(at 133.35 93.98 0)
-		(fields_autoplaced yes)
-		(effects
-			(font
-				(size 1.27 1.27)
-			)
-			(justify left)
-		)
-		(property "Intersheetrefs" "${INTERSHEET_REFS}"
-			(at 143.9552 93.98 0)
-			(effects
-				(font
-					(size 1.27 1.27)
-				)
-				(justify left)
-				(hide yes)
-			)
 		)
 	)
@@
 		)
 	)
-	(global_label "I2C_SCL"
+	(global_label "I2C1_SCL"
+		(shape input)
+		(at 133.35 91.44 0)
+		(fields_autoplaced yes)
+		(effects
+			(font
+				(size 1.27 1.27)
+			)
+			(justify left)
+		)
+		(property "Intersheetrefs" "${INTERSHEET_REFS}"
+			(at 145.1042 91.44 0)
+			(effects
+				(font
+					(size 1.27 1.27)
+				)
+				(justify left)
+				(hide yes)
+			)
+		)
+	)
+	(global_label "I2C1_SDA"
+		(shape input)
+		(at 201.93 49.53 90)
+		(fields_autoplaced yes)
+		(effects
+			(font
+				(size 1.27 1.27)
+			)
+			(justify left)
+		)
+		(property "Intersheetrefs" "${INTERSHEET_REFS}"
+			(at 201.93 37.7153 90)
+			(effects
+				(font
+					(size 1.27 1.27)
+				)
+				(justify left)
+				(hide yes)
+			)
+		)
+	)
+	(global_label "I2C1_SDA"
+		(shape input)
+		(at 133.35 93.98 0)
+		(fields_autoplaced yes)
+		(effects
+			(font
+				(size 1.27 1.27)
+			)
+			(justify left)
+		)
+		(property "Intersheetrefs" "${INTERSHEET_REFS}"
+			(at 145.1647 93.98 0)
+			(effects
+				(font
+					(size 1.27 1.27)
+				)
+				(justify left)
+				(hide yes)
+			)
+		)
+	)
+	(global_label "I2C1_SCL"
 		(shape input)
 		(at 199.39 49.53 90)
@@
 		)
 		(property "Intersheetrefs" "${INTERSHEET_REFS}"
-			(at 199.39 38.9853 90)
-			(effects
-				(font
-					(size 1.27 1.27)
-				)
-				(justify left)
-				(hide yes)
-			)
-		)
-	)
-	(global_label "I2C_SDA"
-		(shape input)
-		(at 201.93 49.53 90)
-		(fields_autoplaced yes)
-		(effects
-			(font
-				(size 1.27 1.27)
-			)
-			(justify left)
-		)
-		(property "Intersheetrefs" "${INTERSHEET_REFS}"
-			(at 201.93 38.9248 90)
-			(effects
-				(font
-					(size 1.27 1.27)
-				)
-				(justify left)
-				(hide yes)
-			)
-		)
-	)
-	(global_label "I2C_SCL"
-		(shape input)
-		(at 133.35 91.44 0)
-		(fields_autoplaced yes)
-		(effects
-			(font
-				(size 1.27 1.27)
-			)
-			(justify left)
-		)
-		(property "Intersheetrefs" "${INTERSHEET_REFS}"
-			(at 143.8947 91.44 0)
+			(at 199.39 37.7758 90)
 			(effects
 				(font
@@
 		(dnp no)
 		(fields_autoplaced yes)
-		(property "Reference" "C27"
+		(property "Reference" "C600"
 			(at 120.65 52.0699 0)
 			(effects
@@
 			(project "rpi_pico_media_board"
 				(path "/883c739e-d2a5-4bc8-a050-29a6043b4072/475bb6c4-6e20-4219-b5f0-3b0e927f6712"
-					(reference "C27")
+					(reference "C600")
 					(unit 1)
 				)
@@
 		(dnp no)
 		(fields_autoplaced yes)
-		(property "Reference" "D10"
+		(property "Reference" "D600"
 			(at 80.01 71.12 0)
 			(effects
@@
 			(project "rpi_pico_media_board"
 				(path "/883c739e-d2a5-4bc8-a050-29a6043b4072/475bb6c4-6e20-4219-b5f0-3b0e927f6712"
-					(reference "D10")
+					(reference "D600")
 					(unit 1)
 				)
@@
 		(on_board yes)
 		(dnp no)
-		(property "Reference" "Y1"
+		(property "Reference" "Y600"
 			(at 65.532 100.33 0)
 			(effects
@@
 			(project "rpi_pico_media_board"
 				(path "/883c739e-d2a5-4bc8-a050-29a6043b4072/475bb6c4-6e20-4219-b5f0-3b0e927f6712"
-					(reference "Y1")
+					(reference "Y600")
 					(unit 1)
 				)
@@
 		(dnp no)
 		(fields_autoplaced yes)
-		(property "Reference" "C28"
+		(property "Reference" "C601"
 			(at 133.35 52.0699 0)
 			(effects
@@
 			(project "rpi_pico_media_board"
 				(path "/883c739e-d2a5-4bc8-a050-29a6043b4072/475bb6c4-6e20-4219-b5f0-3b0e927f6712"
-					(reference "C28")
+					(reference "C601")
 					(unit 1)
 				)
@@
 		(dnp no)
 		(fields_autoplaced yes)
-		(property "Reference" "BT1"
+		(property "Reference" "BT600"
 			(at 56.4515 69.85 90)
 			(effects
@@
 			(project "rpi_pico_media_board"
 				(path "/883c739e-d2a5-4bc8-a050-29a6043b4072/475bb6c4-6e20-4219-b5f0-3b0e927f6712"
-					(reference "BT1")
+					(reference "BT600")
 					(unit 1)
 				)
@@
 		(dnp no)
 		(fields_autoplaced yes)
-		(property "Reference" "R24"
+		(property "Reference" "R600"
 			(at 111.76 81.2799 0)
 			(effects
@@
 			(project "rpi_pico_media_board"
 				(path "/883c739e-d2a5-4bc8-a050-29a6043b4072/475bb6c4-6e20-4219-b5f0-3b0e927f6712"
-					(reference "R24")
+					(reference "R600")
 					(unit 1)
 				)
@@
 		(on_board yes)
 		(dnp no)
-		(property "Reference" "C26"
+		(property "Reference" "C602"
 			(at 51.562 107.95 0)
 			(effects
@@
 			(project "rpi_pico_media_board"
 				(path "/883c739e-d2a5-4bc8-a050-29a6043b4072/475bb6c4-6e20-4219-b5f0-3b0e927f6712"
-					(reference "C26")
+					(reference "C602")
 					(unit 1)
 				)
@@
 		(dnp no)
 		(fields_autoplaced yes)
-		(property "Reference" "R25"
+		(property "Reference" "R601"
 			(at 120.65 81.2799 0)
 			(effects
@@
 			(project "rpi_pico_media_board"
 				(path "/883c739e-d2a5-4bc8-a050-29a6043b4072/475bb6c4-6e20-4219-b5f0-3b0e927f6712"
-					(reference "R25")
+					(reference "R601")
 					(unit 1)
 				)
@@
 		(dnp no)
 		(fields_autoplaced yes)
-		(property "Reference" "U5"
+		(property "Reference" "U600"
 			(at 88.5541 83.82 0)
 			(effects
@@
 			(project "rpi_pico_media_board"
 				(path "/883c739e-d2a5-4bc8-a050-29a6043b4072/475bb6c4-6e20-4219-b5f0-3b0e927f6712"
-					(reference "U5")
+					(reference "U600")
 					(unit 1)
 				)
@@
 		(dnp no)
 		(fields_autoplaced yes)
-		(property "Reference" "D11"
+		(property "Reference" "D601"
 			(at 92.71 71.12 0)
 			(effects
@@
 			(project "rpi_pico_media_board"
 				(path "/883c739e-d2a5-4bc8-a050-29a6043b4072/475bb6c4-6e20-4219-b5f0-3b0e927f6712"
-					(reference "D11")
+					(reference "D601")
 					(unit 1)
 				)
@@
 		(dnp no)
 		(fields_autoplaced yes)
-		(property "Reference" "Brd1"
+		(property "Reference" "Brd600"
 			(at 205.74 60.9599 0)
 			(effects
@@
 			(project ""
 				(path "/883c739e-d2a5-4bc8-a050-29a6043b4072/475bb6c4-6e20-4219-b5f0-3b0e927f6712"
-					(reference "Brd1")
+					(reference "Brd600")
 					(unit 1)
 				)

Commit message: Minor BOM updates
Parts:
- C600: Manufacturer Product Number CL21A106KOQNNNE -> (none)
- C601: Manufacturer Product Number CL10B104KB8NNNC -> (none)
- C602: Manufacturer Product Number CL10C150JB8NNNC -> (none)
Changed lines of the file:
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@@
 			)
 		)
-		(property "Manufacturer Product Number" "CL21A106KOQNNNE"
+		(property "Manufacturer Product Number" ""
 			(at 116.84 53.34 0)
 			(effects
@@
 			)
 		)
-		(property "Manufacturer Product Number" "CL10B104KB8NNNC"
+		(property "Manufacturer Product Number" ""
 			(at 129.54 53.34 0)
 			(effects
@@
 			)
 		)
-		(property "Manufacturer Product Number" "CL10C150JB8NNNC"
+		(property "Manufacturer Product Number" ""
 			(at 50.8 110.49 0)
 			(effects

Commit message: DRC cleanup
Parts:
- D600, D601: Manufacturer Product Number 1N4148W -> (none)
- R600, R601: Manufacturer Product Number 0805W8F5101T5E -> (none)
- U600: Manufacturer Product Number PCF8563TS/5,118 -> (none)
- Y600: Manufacturer Product Number OK2EL89CJI-111YLC-32.768K -> (none)
Changed lines of the file:
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@@
 			)
 		)
-		(property "Manufacturer Product Number" "1N4148W"
+		(property "Manufacturer Product Number" ""
 			(at 80.01 77.47 0)
 			(effects
@@
 			)
 		)
-		(property "Manufacturer Product Number" "OK2EL89CJI-111YLC-32.768K"
+		(property "Manufacturer Product Number" ""
 			(at 63.5 105.41 0)
 			(effects
@@
 			)
 		)
-		(property "Manufacturer Product Number" "0805W8F5101T5E"
+		(property "Manufacturer Product Number" ""
 			(at 109.22 82.55 0)
 			(effects
@@
 			)
 		)
-		(property "Manufacturer Product Number" "0805W8F5101T5E"
+		(property "Manufacturer Product Number" ""
 			(at 118.11 82.55 0)
 			(effects
@@
 			)
 		)
-		(property "Manufacturer Product Number" "PCF8563TS/5,118"
+		(property "Manufacturer Product Number" ""
 			(at 86.36 96.52 0)
 			(effects
@@
 			)
 		)
-		(property "Manufacturer Product Number" "1N4148W"
+		(property "Manufacturer Product Number" ""
 			(at 92.71 77.47 0)
 			(effects
