File: HW/rpi_pico_media_board/[5]Macro_Pad.kicad_sch (KiCad schematic)
At the start: 12 parts

Commit message: Scheme improvements
Parts:
- added C500, C501, C502: 100nF, Capacitor_SMD:C_0603_1608Metric, symbol Device:C
- added D500, D501, D502, D503, D504, D505, D506, D507, D508, D509, D510, D511: 1N4148, Diode_SMD:D_SOD-123, symbol Device:D
- added D512, D513, D514: LED, LED_SMD:LED_0603_1608Metric, symbol Device:LED
- added Q500, Q501, Q502: T2N7002AK, Package_TO_SOT_SMD:SOT-23, symbol Transistor_FET:T2N7002AK
- added R500, R501, R502, R503: 22R, Resistor_SMD:R_0603_1608Metric, symbol Device:R
- added R504, R505, R506: 0R, Resistor_SMD:R_0603_1608Metric, symbol Device:R
- added R507, R509, R511: 510R, Resistor_SMD:R_0402_1005Metric, symbol Device:R
- added R508, R510, R512: 12kR, Resistor_SMD:R_0402_1005Metric, symbol Device:R
- renumbered SW1 to SW500, SW2 to SW501, SW3 to SW502, SW4 to SW503, SW5 to SW504, SW6 to SW505, SW7 to SW506, SW8 to SW507, SW9 to SW508, SW10 to SW509, SW11 to SW510, SW12 to SW511
Connections:
- net at SW506.1: now also SW502.1, SW510.1, R501.2
- net at SW506.2: now also D506.2 (A)
- net at SW511.1: now also SW503.1, SW507.1, R500.2
- net at SW511.2: now also D511.2 (A)
- net at SW509.1: now also SW501.1, SW505.1, R502.2
- net at SW509.2: now also D509.2 (A)
- net at SW508.1: now also SW500.1, SW504.1, R503.2
- net at SW508.2: now also D508.2 (A)
- net at SW510.2: now also D510.2 (A)
- net at SW500.2: now also D500.2 (A)
- net at SW502.2: now also D502.2 (A)
- net at SW507.2: now also D507.2 (A)
- net at SW504.2: now also D504.2 (A)
- net at SW505.2: now also D505.2 (A)
- net at SW501.2: now also D501.2 (A)
- net at SW503.2: now also D503.2 (A)
- new net: D508.1 (K), D509.1 (K), D510.1 (K), D511.1 (K), R506.2
- new net: Q500.1 (G), R508.1
- new net: Q502.1 (G), R512.1
- new net: D500.1 (K), D501.1 (K), D502.1 (K), D503.1 (K), R504.2
- new net: D504.1 (K), D505.1 (K), D506.1 (K), D507.1 (K), R505.2
- new net: Q501.1 (G), R510.1
- new net +5V: R507.2, R509.2, R511.2
- new net GND: C500.2, C501.2, C502.2, Q500.2 (S), Q501.2 (S), Q502.2 (S)
- new net MACRO_PAD_BTN_COL_0: R503.1
- new net MACRO_PAD_BTN_COL_1: R502.1
- new net MACRO_PAD_BTN_COL_2: R501.1
- new net MACRO_PAD_BTN_COL_3: R500.1
- new net MACRO_PAD_BTN_ROW_0: C500.1, R504.1
- new net MACRO_PAD_BTN_ROW_1: C501.1, R505.1
- new net MACRO_PAD_BTN_ROW_2: C502.1, R506.1
- new net USR_LED_0: R508.2
- new net USR_LED_0_A: D512.2 (A), R507.1
- new net USR_LED_0_K: D512.1 (K), Q500.3 (D)
- new net USR_LED_1: R510.2
- new net USR_LED_1_A: D513.2 (A), R509.1
- new net USR_LED_1_K: D513.1 (K), Q501.3 (D)
- new net USR_LED_2: R512.2
- new net USR_LED_2_A: D514.2 (A), R511.1
- new net USR_LED_2_K: D514.1 (K), Q502.3 (D)
Other:
- note added: "[5]Macro Pad"
- moved on the sheet: SW500, SW501, SW502, SW503, SW504, SW505, SW506, SW507, SW508, SW509, SW510, SW511

Commit message: Minor BOM updates
Parts:
- C500, C501, C502: Manufacturer Product Number CL10B104KB8NNNC -> (none)
- D512, D513, D514: Manufacturer (none) -> XINGLIGHT; Manufacturer Part Number (none) -> XL-1608SURC-06; Manufacturer_Name XINGLIGHT -> (none); Manufacturer_Part_Number XL-1608SURC-06 -> (none)
- Q500, Q501, Q502: Manufacturer (none) -> TOSHIBA; Manufacturer Part Number (none) -> T2N7002AK,LM; Manufacturer_Name TOSHIBA -> (none); Manufacturer_Part_Number T2N7002AK,LM -> (none)
Changed lines of the file:
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@@
 	)
 	(symbol
-		(lib_name "rpi_pico_media_board:SW_PUSH_6mm_H5mm")
 		(lib_id "rpi_pico_media_board:SW_PUSH_6mm_H5mm")
 		(at 120.65 85.09 0)
@@
 			)
 		)
-		(property "Manufacturer_Name" "TOSHIBA"
+		(property "Manufacturer_Name" ""
 			(at 186.69 90.17 0)
 			(effects
@@
 			)
 		)
-		(property "Manufacturer_Part_Number" "T2N7002AK,LM"
+		(property "Manufacturer_Part_Number" ""
+			(at 186.69 90.17 0)
+			(effects
+				(font
+					(size 1.27 1.27)
+				)
+				(hide yes)
+			)
+		)
+		(property "Manufacturer" "TOSHIBA"
+			(at 186.69 90.17 0)
+			(effects
+				(font
+					(size 1.27 1.27)
+				)
+				(hide yes)
+			)
+		)
+		(property "Manufacturer Part Number" "T2N7002AK,LM"
 			(at 186.69 90.17 0)
 			(effects
@@
 	)
 	(symbol
-		(lib_name "rpi_pico_media_board:SW_PUSH_6mm_H5mm")
 		(lib_id "rpi_pico_media_board:SW_PUSH_6mm_H5mm")
 		(at 146.05 110.49 0)
@@
 			)
 		)
-		(property "Manufacturer Product Number" "CL10B104KB8NNNC"
+		(property "Manufacturer Product Number" ""
 			(at 44.45 134.62 0)
 			(effects
@@
 	)
 	(symbol
-		(lib_name "rpi_pico_media_board:SW_PUSH_6mm_H5mm")
 		(lib_id "rpi_pico_media_board:SW_PUSH_6mm_H5mm")
 		(at 95.25 110.49 0)
@@
 	)
 	(symbol
-		(lib_name "rpi_pico_media_board:SW_PUSH_6mm_H5mm")
 		(lib_id "rpi_pico_media_board:SW_PUSH_6mm_H5mm")
 		(at 69.85 110.49 0)
@@
 	)
 	(symbol
-		(lib_name "rpi_pico_media_board:SW_PUSH_6mm_H5mm")
 		(lib_id "rpi_pico_media_board:SW_PUSH_6mm_H5mm")
 		(at 120.65 110.49 0)
@@
 	)
 	(symbol
-		(lib_name "rpi_pico_media_board:SW_PUSH_6mm_H5mm")
 		(lib_id "rpi_pico_media_board:SW_PUSH_6mm_H5mm")
 		(at 69.85 59.69 0)
@@
 			)
 		)
-		(property "Manufacturer Product Number" "CL10B104KB8NNNC"
+		(property "Manufacturer Product Number" ""
 			(at 44.45 109.22 0)
 			(effects
@@
 			)
 		)
-		(property "Manufacturer_Name" "XINGLIGHT"
+		(property "Manufacturer_Name" ""
+			(at 184.15 77.47 0)
+			(effects
+				(font
+					(size 1.27 1.27)
+				)
+				(hide yes)
+			)
+		)
+		(property "Manufacturer_Part_Number" ""
 			(at 184.15 77.47 0)
 			(effects
@@
 			)
 		)
-		(property "Manufacturer_Part_Number" "XL-1608SURC-06"
+		(property "Manufacturer" "XINGLIGHT"
+			(at 184.15 77.47 0)
+			(effects
+				(font
+					(size 1.27 1.27)
+				)
+				(hide yes)
+			)
+		)
+		(property "Manufacturer Part Number" "XL-1608SURC-06"
 			(at 184.15 77.47 0)
 			(effects
@@
 	)
 	(symbol
-		(lib_name "rpi_pico_media_board:SW_PUSH_6mm_H5mm")
 		(lib_id "rpi_pico_media_board:SW_PUSH_6mm_H5mm")
 		(at 120.65 59.69 0)
@@
 			)
 		)
-		(property "Manufacturer_Name" "XINGLIGHT"
+		(property "Manufacturer_Name" ""
+			(at 250.19 77.47 0)
+			(effects
+				(font
+					(size 1.27 1.27)
+				)
+				(hide yes)
+			)
+		)
+		(property "Manufacturer_Part_Number" ""
+			(at 250.19 77.47 0)
+			(effects
+				(font
+					(size 1.27 1.27)
+				)
+				(hide yes)
+			)
+		)
+		(property "Manufacturer" "XINGLIGHT"
 			(at 250.19 77.47 0)
 			(effects
@@
 			)
 		)
-		(property "Manufacturer_Part_Number" "XL-1608SURC-06"
+		(property "Manufacturer Part Number" "XL-1608SURC-06"
 			(at 250.19 77.47 0)
 			(effects
@@
 			)
 		)
-		(property "Manufacturer_Name" "XINGLIGHT"
+		(property "Manufacturer_Name" ""
 			(at 217.17 77.47 0)
 			(effects
@@
 			)
 		)
-		(property "Manufacturer_Part_Number" "XL-1608SURC-06"
+		(property "Manufacturer_Part_Number" ""
+			(at 217.17 77.47 0)
+			(effects
+				(font
+					(size 1.27 1.27)
+				)
+				(hide yes)
+			)
+		)
+		(property "Manufacturer" "XINGLIGHT"
+			(at 217.17 77.47 0)
+			(effects
+				(font
+					(size 1.27 1.27)
+				)
+				(hide yes)
+			)
+		)
+		(property "Manufacturer Part Number" "XL-1608SURC-06"
 			(at 217.17 77.47 0)
 			(effects
@@
 	)
 	(symbol
-		(lib_name "rpi_pico_media_board:SW_PUSH_6mm_H5mm")
 		(lib_id "rpi_pico_media_board:SW_PUSH_6mm_H5mm")
 		(at 146.05 85.09 0)
@@
 			)
 		)
-		(property "Manufacturer Product Number" "CL10B104KB8NNNC"
+		(property "Manufacturer Product Number" ""
 			(at 44.45 83.82 0)
 			(effects
@@
 			)
 		)
-		(property "Manufacturer_Name" "TOSHIBA"
+		(property "Manufacturer_Name" ""
+			(at 219.71 90.17 0)
+			(effects
+				(font
+					(size 1.27 1.27)
+				)
+				(hide yes)
+			)
+		)
+		(property "Manufacturer_Part_Number" ""
 			(at 219.71 90.17 0)
 			(effects
@@
 			)
 		)
-		(property "Manufacturer_Part_Number" "T2N7002AK,LM"
+		(property "Manufacturer" "TOSHIBA"
+			(at 219.71 90.17 0)
+			(effects
+				(font
+					(size 1.27 1.27)
+				)
+				(hide yes)
+			)
+		)
+		(property "Manufacturer Part Number" "T2N7002AK,LM"
 			(at 219.71 90.17 0)
 			(effects
@@
 	)
 	(symbol
-		(lib_name "rpi_pico_media_board:SW_PUSH_6mm_H5mm")
 		(lib_id "rpi_pico_media_board:SW_PUSH_6mm_H5mm")
 		(at 69.85 85.09 0)
@@
 	)
 	(symbol
-		(lib_name "rpi_pico_media_board:SW_PUSH_6mm_H5mm")
 		(lib_id "rpi_pico_media_board:SW_PUSH_6mm_H5mm")
 		(at 95.25 85.09 0)
@@
 	)
 	(symbol
-		(lib_name "rpi_pico_media_board:SW_PUSH_6mm_H5mm")
 		(lib_id "rpi_pico_media_board:SW_PUSH_6mm_H5mm")
 		(at 95.25 59.69 0)
@@
 			)
 		)
-		(property "Manufacturer_Name" "TOSHIBA"
+		(property "Manufacturer_Name" ""
+			(at 252.73 90.17 0)
+			(effects
+				(font
+					(size 1.27 1.27)
+				)
+				(hide yes)
+			)
+		)
+		(property "Manufacturer_Part_Number" ""
+			(at 252.73 90.17 0)
+			(effects
+				(font
+					(size 1.27 1.27)
+				)
+				(hide yes)
+			)
+		)
+		(property "Manufacturer" "TOSHIBA"
 			(at 252.73 90.17 0)
 			(effects
@@
 			)
 		)
-		(property "Manufacturer_Part_Number" "T2N7002AK,LM"
+		(property "Manufacturer Part Number" "T2N7002AK,LM"
 			(at 252.73 90.17 0)
 			(effects
@@
 	)
 	(symbol
-		(lib_name "rpi_pico_media_board:SW_PUSH_6mm_H5mm")
 		(lib_id "rpi_pico_media_board:SW_PUSH_6mm_H5mm")
 		(at 146.05 59.69 0)

Commit message: DRC cleanup
Parts:
- D500, D501, D502, D503, D504, D505, D506, D507, D508, D509, D510, D511: Manufacturer Product Number 1N4148W -> (none)
- R504, R505, R506: Manufacturer Part Number 0603WAF220JT5E -> 0603WAF0000T5E
- R507, R509, R511: footprint Resistor_SMD:R_0402_1005Metric -> Resistor_SMD:R_0603_1608Metric; Manufacturer (none) -> UNI-ROYAL(Uniroyal Elec); Manufacturer Part Number (none) -> 0603WAF5100T5E; Manufacturer_Name UNI-ROYAL(Uniroyal Elec) -> (none); Manufacturer_Part_Number 0402WGF5100TCE -> (none)
- R508, R510, R512: footprint Resistor_SMD:R_0402_1005Metric -> Resistor_SMD:R_0603_1608Metric; Manufacturer (none) -> UNI-ROYAL(Uniroyal Elec); Manufacturer Part Number (none) -> 0603WAF1202T5E; Manufacturer_Name UNI-ROYAL(Uniroyal Elec) -> (none); Manufacturer_Part_Number 0402WGF1202TCE -> (none)
- U500: renamed from SW500; value ~ -> SW
- U501: renamed from SW501; value ~ -> SW
- U502: renamed from SW502; value ~ -> SW
- U503: renamed from SW503; value ~ -> SW
- U504: renamed from SW504; value ~ -> SW
- U505: renamed from SW505; value ~ -> SW
- U506: renamed from SW506; value ~ -> SW
- U507: renamed from SW507; value ~ -> SW
- U508: renamed from SW508; value ~ -> SW
- U509: renamed from SW509; value ~ -> SW
- U510: renamed from SW510; value ~ -> SW
- U511: renamed from SW511; value ~ -> SW
