File: HW/rpi_pico_media_board/[3]PCM5102.kicad_sch (KiCad schematic)
At the start: 22 parts, among them J2 AudioJack3_Ground_SwitchTR, J3 Conn_01x03_Pin, J4 Conn_01x05_Pin, U4 PCM5102A

Commit message: Scheme improvements
Parts:
- removed J4: Conn_01x05_Pin, Connector_PinHeader_2.54mm:PinHeader_1x05_P2.54mm_Vertical, symbol Connector_Generic:Conn_01x05
- renumbered C14 to C300, C15 to C301, C16 to C302, C17 to C303, C18 to C304, C21 to C305, C19 to C306, C22 to C307, C20 to C308, C23 to C309, C12 to C310, C13 to C311, J2 to J300, J3 to J301, R14 to R300, R15 to R301, R16 to R302, R17 to R303, R12 to R304, R13 to R305, U4 to U300
Connections:
- net I2S3_CK renamed I2S_PCM5102_SCK
- net I2S3_SD renamed I2S_PCM5102_DATA
- net I2S3_WS renamed I2S_PCM5102_SCL
Other:
- note added: "[3]PCM5102"
- note removed: "I2S Connector"

Commit message: DRC cleanup
Parts:
- added R304, R305, R306, R307: 22R, Resistor_SMD:R_0603_1608Metric, symbol Device:R
- renumbered R304 to R308, R305 to R309
Connections:
- net +3.3V: now also R306.1; no longer U300.17 (XSMT)
- net GND: now also R304.1, R305.1, R307.1; no longer U300.10 (DEMP), U300.11 (FLT), U300.16 (FMT)
- new net DEMP: R305.2, U300.10 (DEMP)
- new net FLT: R304.2, U300.11 (FLT)
- new net FMT: R307.2, U300.16 (FMT)
- new net XSMT: R306.2, U300.17 (XSMT)

Commit message: Very initial PCB layout
Connections:
- net +3.3VA renamed +3.3VA_PCM
Changed lines of the file:
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@@
 	)
 	(junction
-		(at 152.4 91.44)
+		(at 187.96 41.91)
 		(diameter 0)
 		(color 0 0 0 0)
 	)
 	(junction
-		(at 187.96 72.39)
+		(at 152.4 91.44)
 		(diameter 0)
 		(color 0 0 0 0)
 	)
 	(junction
-		(at 187.96 41.91)
+		(at 187.96 72.39)
 		(diameter 0)
 		(color 0 0 0 0)
@@
 	)
 	(junction
-		(at 187.96 60.96)
-		(diameter 0)
-		(color 0 0 0 0)
-	)
-	(junction
 		(at 187.96 80.01)
 		(diameter 0)
@@
 	)
 	(junction
+		(at 187.96 60.96)
+		(diameter 0)
+		(color 0 0 0 0)
+	)
+	(junction
 		(at 143.51 78.74)
 		(diameter 0)
@@
 	(wire
 		(pts
+			(xy 187.96 41.91) (xy 195.58 41.91)
+		)
+		(stroke
+			(width 0)
+			(type default)
+		)
+	)
+	(wire
+		(pts
 			(xy 195.58 53.34) (xy 195.58 50.8)
 		)
@@
 	(wire
 		(pts
+			(xy 187.96 60.96) (xy 195.58 60.96)
+		)
+		(stroke
+			(width 0)
+			(type default)
+		)
+	)
+	(wire
+		(pts
 			(xy 128.27 66.04) (xy 134.62 66.04)
 		)
@@
 	(wire
 		(pts
-			(xy 187.96 41.91) (xy 195.58 41.91)
-		)
-		(stroke
-			(width 0)
-			(type default)
-		)
-	)
-	(wire
-		(pts
 			(xy 179.07 72.39) (xy 179.07 69.85)
 		)
@@
 	(wire
 		(pts
-			(xy 187.96 60.96) (xy 195.58 60.96)
+			(xy 179.07 60.96) (xy 187.96 60.96)
 		)
 		(stroke
@@
 	(wire
 		(pts
-			(xy 179.07 60.96) (xy 187.96 60.96)
-		)
-		(stroke
-			(width 0)
-			(type default)
-		)
-	)
-	(wire
-		(pts
 			(xy 115.57 44.45) (xy 171.45 44.45)
 		)
@@
 	)
 	(symbol
-		(lib_id "power:+3.3VA")
-		(at 187.96 60.96 0)
-		(unit 1)
-		(exclude_from_sim no)
-		(in_bom yes)
-		(on_board yes)
-		(dnp no)
-		(property "Reference" "#PWR28"
-			(at 187.96 64.77 0)
-			(effects
-				(font
-					(size 1.27 1.27)
-				)
-				(hide yes)
-			)
-		)
-		(property "Value" "+3.3VA"
-			(at 192.532 59.182 0)
-			(effects
-				(font
-					(size 1.27 1.27)
-				)
-			)
-		)
-		(property "Footprint" ""
-			(at 187.96 60.96 0)
-			(effects
-				(font
-					(size 1.27 1.27)
-				)
-				(hide yes)
-			)
-		)
-		(property "Datasheet" ""
-			(at 187.96 60.96 0)
-			(effects
-				(font
-					(size 1.27 1.27)
-				)
-				(hide yes)
-			)
-		)
-		(property "Description" "Power symbol creates a global label with name \"+3.3VA\""
-			(at 187.96 60.96 0)
-			(effects
-				(font
-					(size 1.27 1.27)
-				)
-				(hide yes)
-			)
-		)
-		(pin "1"
-		)
-		(instances
-			(project "rpi_pico_media_board"
-				(path "/883c739e-d2a5-4bc8-a050-29a6043b4072/373bacf3-831c-41f0-9f95-7ac0a975261a"
-					(reference "#PWR28")
-					(unit 1)
-				)
-			)
-		)
-	)
-	(symbol
 		(lib_id "Device:R")
 		(at 88.9 76.2 90)
@@
 	)
 	(symbol
+		(lib_id "power:+3.3VA")
+		(at 187.96 60.96 0)
+		(unit 1)
+		(exclude_from_sim no)
+		(in_bom yes)
+		(on_board yes)
+		(dnp no)
+		(property "Reference" "#PWR28"
+			(at 187.96 64.77 0)
+			(effects
+				(font
+					(size 1.27 1.27)
+				)
+				(hide yes)
+			)
+		)
+		(property "Value" "+3.3VA_PCM"
+			(at 187.96 57.15 0)
+			(effects
+				(font
+					(size 1.27 1.27)
+				)
+			)
+		)
+		(property "Footprint" ""
+			(at 187.96 60.96 0)
+			(effects
+				(font
+					(size 1.27 1.27)
+				)
+				(hide yes)
+			)
+		)
+		(property "Datasheet" ""
+			(at 187.96 60.96 0)
+			(effects
+				(font
+					(size 1.27 1.27)
+				)
+				(hide yes)
+			)
+		)
+		(property "Description" "Power symbol creates a global label with name \"+3.3VA\""
+			(at 187.96 60.96 0)
+			(effects
+				(font
+					(size 1.27 1.27)
+				)
+				(hide yes)
+			)
+		)
+		(pin "1"
+		)
+		(instances
+			(project "rpi_pico_media_board"
+				(path "/883c739e-d2a5-4bc8-a050-29a6043b4072/373bacf3-831c-41f0-9f95-7ac0a975261a"
+					(reference "#PWR28")
+					(unit 1)
+				)
+			)
+		)
+	)
+	(symbol
+		(lib_id "power:+3.3VA")
+		(at 187.96 41.91 0)
+		(unit 1)
+		(exclude_from_sim no)
+		(in_bom yes)
+		(on_board yes)
+		(dnp no)
+		(property "Reference" "#PWR26"
+			(at 187.96 45.72 0)
+			(effects
+				(font
+					(size 1.27 1.27)
+				)
+				(hide yes)
+			)
+		)
+		(property "Value" "+3.3VA_PCM"
+			(at 187.96 38.1 0)
+			(effects
+				(font
+					(size 1.27 1.27)
+				)
+			)
+		)
+		(property "Footprint" ""
+			(at 187.96 41.91 0)
+			(effects
+				(font
+					(size 1.27 1.27)
+				)
+				(hide yes)
+			)
+		)
+		(property "Datasheet" ""
+			(at 187.96 41.91 0)
+			(effects
+				(font
+					(size 1.27 1.27)
+				)
+				(hide yes)
+			)
+		)
+		(property "Description" "Power symbol creates a global label with name \"+3.3VA\""
+			(at 187.96 41.91 0)
+			(effects
+				(font
+					(size 1.27 1.27)
+				)
+				(hide yes)
+			)
+		)
+		(pin "1"
+		)
+		(instances
+			(project "rpi_pico_media_board"
+				(path "/883c739e-d2a5-4bc8-a050-29a6043b4072/373bacf3-831c-41f0-9f95-7ac0a975261a"
+					(reference "#PWR26")
+					(unit 1)
+				)
+			)
+		)
+	)
+	(symbol
 		(lib_id "Device:C")
 		(at 134.62 85.09 0)
@@
 					(unit 1)
 				)
-			)
-		)
-	)
-	(symbol
-		(lib_id "power:+3.3VA")
-		(at 187.96 41.91 0)
-		(unit 1)
-		(exclude_from_sim no)
-		(in_bom yes)
-		(on_board yes)
-		(dnp no)
-		(property "Reference" "#PWR26"
-			(at 187.96 45.72 0)
-			(effects
-				(font
-					(size 1.27 1.27)
-				)
-				(hide yes)
-			)
-		)
-		(property "Value" "+3.3VA"
-			(at 192.532 40.132 0)
-			(effects
-				(font
-					(size 1.27 1.27)
-				)
-			)
-		)
-		(property "Footprint" ""
-			(at 187.96 41.91 0)
-			(effects
-				(font
-					(size 1.27 1.27)
-				)
-				(hide yes)
-			)
-		)
-		(property "Datasheet" ""
-			(at 187.96 41.91 0)
-			(effects
-				(font
-					(size 1.27 1.27)
-				)
-				(hide yes)
-			)
-		)
-		(property "Description" "Power symbol creates a global label with name \"+3.3VA\""
-			(at 187.96 41.91 0)
-			(effects
-				(font
-					(size 1.27 1.27)
-				)
-				(hide yes)
-			)
-		)
-		(pin "1"
-		)
-		(instances
-			(project "rpi_pico_media_board"
-				(path "/883c739e-d2a5-4bc8-a050-29a6043b4072/373bacf3-831c-41f0-9f95-7ac0a975261a"
-					(reference "#PWR26")
-					(unit 1)
-				)
