File: KiCad/[1]Power.kicad_sch (KiCad schematic)
At the start: 29 parts, among them J100 Barrel_Jack_Switch_Pin3Ring, Q100 T2N7002AK, U100 HT7533-1, U101 HT7533-1

Commit message: Manufacture files preparation
Parts:
- J100: Manufacturer (none) -> SHOU HAN; Manufacturer Part Number (none) -> DC005
- L100: Manufacturer Part Number LQG18HN10NJ00D -> LQW18AN10NG10D
- L101: Manufacturer Part Number LQM2HPN2R2MG0L -> DFE252012F-2R2M=P2
- PS100: Manufacturer Silergy -> Silergy Corp
