File: KiCad/[3]PCM5102.kicad_sch (KiCad schematic)
At the start: 25 parts, among them J300 AudioJack3_Ground_SwitchTR, J301 Conn_01x03_Pin, U300 PCM5102A

Commit message: Manufacture files preparation
Parts:
- C302, C304, C306, C308: Manufacturer Part Number CL10B104KB8NNNC -> CL10B104KA8NNNC
- J300: Manufacturer (none) -> SHOU HAN; Manufacturer Part Number (none) -> PJ-342
- J301: now not fitted
- U300: Manufacturer Part Number PCM5102APWR -> PCM5102AQPWRQ1
Changed lines of the file:
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@@
 			)
 		)
-		(property "Manufacturer Part Number" "CL10B104KB8NNNC"
+		(property "Manufacturer Part Number" "CL10B104KA8NNNC"
 			(at 143.51 85.09 0)
 			(effects
@@
 		(dnp no)
 		(fields_autoplaced yes)
-		(property "Reference" "#PWR18"
+		(property "Reference" "#PWR018"
 			(at 87.63 168.91 0)
 			(effects
@@
 			(project "rpi_pico_media_board"
 				(path "/883c739e-d2a5-4bc8-a050-29a6043b4072/373bacf3-831c-41f0-9f95-7ac0a975261a"
-					(reference "#PWR18")
+					(reference "#PWR018")
 					(unit 1)
 				)
@@
 		(dnp no)
 		(fields_autoplaced yes)
-		(property "Reference" "#PWR19"
+		(property "Reference" "#PWR019"
 			(at 80.01 91.44 0)
 			(effects
@@
 			(project "rpi_pico_media_board"
 				(path "/883c739e-d2a5-4bc8-a050-29a6043b4072/373bacf3-831c-41f0-9f95-7ac0a975261a"
-					(reference "#PWR19")
+					(reference "#PWR019")
 					(unit 1)
 				)
@@
 			)
 		)
-		(property "Manufacturer Part Number" "CL10B104KB8NNNC"
+		(property "Manufacturer Part Number" "CL10B104KA8NNNC"
 			(at 179.07 46.99 0)
 			(effects
@@
 		(on_board yes)
 		(dnp no)
-		(property "Reference" "#PWR30"
+		(property "Reference" "#PWR030"
 			(at 187.96 83.82 0)
 			(effects
@@
 			(project "rpi_pico_media_board"
 				(path "/883c739e-d2a5-4bc8-a050-29a6043b4072/373bacf3-831c-41f0-9f95-7ac0a975261a"
-					(reference "#PWR30")
+					(reference "#PWR030")
 					(unit 1)
 				)
@@
 		(dnp no)
 		(fields_autoplaced yes)
-		(property "Reference" "#PWR15"
+		(property "Reference" "#PWR015"
 			(at 68.58 78.74 0)
 			(effects
@@
 			(project "rpi_pico_media_board"
 				(path "/883c739e-d2a5-4bc8-a050-29a6043b4072/373bacf3-831c-41f0-9f95-7ac0a975261a"
-					(reference "#PWR15")
+					(reference "#PWR015")
 					(unit 1)
 				)
@@
 		(on_board yes)
 		(dnp no)
-		(property "Reference" "#PWR28"
+		(property "Reference" "#PWR028"
 			(at 187.96 64.77 0)
 			(effects
@@
 			(project "rpi_pico_media_board"
 				(path "/883c739e-d2a5-4bc8-a050-29a6043b4072/373bacf3-831c-41f0-9f95-7ac0a975261a"
-					(reference "#PWR28")
+					(reference "#PWR028")
 					(unit 1)
 				)
@@
 		(on_board yes)
 		(dnp no)
-		(property "Reference" "#PWR26"
+		(property "Reference" "#PWR026"
 			(at 187.96 45.72 0)
 			(effects
@@
 			(project "rpi_pico_media_board"
 				(path "/883c739e-d2a5-4bc8-a050-29a6043b4072/373bacf3-831c-41f0-9f95-7ac0a975261a"
-					(reference "#PWR26")
+					(reference "#PWR026")
 					(unit 1)
 				)
@@
 		(dnp no)
 		(fields_autoplaced yes)
-		(property "Reference" "#PWR24"
+		(property "Reference" "#PWR024"
 			(at 168.91 138.43 0)
 			(effects
@@
 			(project "rpi_pico_media_board"
 				(path "/883c739e-d2a5-4bc8-a050-29a6043b4072/373bacf3-831c-41f0-9f95-7ac0a975261a"
-					(reference "#PWR24")
+					(reference "#PWR024")
 					(unit 1)
 				)
@@
 		(dnp no)
 		(fields_autoplaced yes)
-		(property "Reference" "#PWR22"
+		(property "Reference" "#PWR022"
 			(at 152.4 97.79 0)
 			(effects
@@
 			(project "rpi_pico_media_board"
 				(path "/883c739e-d2a5-4bc8-a050-29a6043b4072/373bacf3-831c-41f0-9f95-7ac0a975261a"
-					(reference "#PWR22")
+					(reference "#PWR022")
 					(unit 1)
 				)
@@
 		(dnp no)
 		(fields_autoplaced yes)
-		(property "Reference" "#PWR25"
+		(property "Reference" "#PWR025"
 			(at 180.34 146.05 0)
 			(effects
@@
 			(project "rpi_pico_media_board"
 				(path "/883c739e-d2a5-4bc8-a050-29a6043b4072/373bacf3-831c-41f0-9f95-7ac0a975261a"
-					(reference "#PWR25")
+					(reference "#PWR025")
 					(unit 1)
 				)
@@
 			)
 		)
-		(property "Manufacturer Part Number" "CL10B104KB8NNNC"
+		(property "Manufacturer Part Number" "CL10B104KA8NNNC"
 			(at 179.07 66.04 0)
 			(effects
@@
 			)
 		)
-		(property "Manufacturer Part Number" "CL10B104KB8NNNC"
+		(property "Manufacturer Part Number" "CL10B104KA8NNNC"
 			(at 179.07 85.09 0)
 			(effects
@@
 		(dnp no)
 		(fields_autoplaced yes)
-		(property "Reference" "#PWR17"
+		(property "Reference" "#PWR017"
 			(at 87.63 138.43 0)
 			(effects
@@
 			(project "rpi_pico_media_board"
 				(path "/883c739e-d2a5-4bc8-a050-29a6043b4072/373bacf3-831c-41f0-9f95-7ac0a975261a"
-					(reference "#PWR17")
+					(reference "#PWR017")
 					(unit 1)
 				)
@@
 		(dnp no)
 		(fields_autoplaced yes)
-		(property "Reference" "#PWR20"
+		(property "Reference" "#PWR020"
 			(at 115.57 97.79 0)
 			(effects
@@
 			(project "rpi_pico_media_board"
 				(path "/883c739e-d2a5-4bc8-a050-29a6043b4072/373bacf3-831c-41f0-9f95-7ac0a975261a"
-					(reference "#PWR20")
+					(reference "#PWR020")
 					(unit 1)
 				)
@@
 			)
 		)
-		(property "Manufacturer" ""
+		(property "Manufacturer" "SHOU HAN"
 			(at 156.21 128.27 0)
 			(effects
@@
 			)
 		)
+		(property "Manufacturer Part Number" "PJ-342"
+			(at 156.21 128.27 0)
+			(effects
+				(font
+					(size 1.27 1.27)
+				)
+				(hide yes)
+			)
+		)
 		(pin "RN"
 		)
@@
 			)
 		)
-		(property "Manufacturer Part Number" "PCM5102APWR"
+		(property "Manufacturer Part Number" "PCM5102AQPWRQ1"
 			(at 115.57 68.58 0)
 			(effects
@@
 		(on_board yes)
 		(dnp no)
-		(property "Reference" "#PWR16"
+		(property "Reference" "#PWR016"
 			(at 74.93 77.47 0)
 			(effects
@@
 			(project "rpi_pico_media_board"
 				(path "/883c739e-d2a5-4bc8-a050-29a6043b4072/373bacf3-831c-41f0-9f95-7ac0a975261a"
-					(reference "#PWR16")
+					(reference "#PWR016")
 					(unit 1)
 				)
@@
 		(on_board yes)
 		(dnp no)
-		(property "Reference" "#PWR31"
+		(property "Reference" "#PWR031"
 			(at 187.96 97.79 0)
 			(effects
@@
 			(project "rpi_pico_media_board"
 				(path "/883c739e-d2a5-4bc8-a050-29a6043b4072/373bacf3-831c-41f0-9f95-7ac0a975261a"
-					(reference "#PWR31")
+					(reference "#PWR031")
 					(unit 1)
 				)
@@
 		(on_board yes)
 		(dnp no)
-		(property "Reference" "#PWR29"
+		(property "Reference" "#PWR029"
 			(at 187.96 78.74 0)
 			(effects
@@
 			(project "rpi_pico_media_board"
 				(path "/883c739e-d2a5-4bc8-a050-29a6043b4072/373bacf3-831c-41f0-9f95-7ac0a975261a"
-					(reference "#PWR29")
+					(reference "#PWR029")
 					(unit 1)
 				)
@@
 		(on_board yes)
 		(dnp no)
-		(property "Reference" "#PWR27"
+		(property "Reference" "#PWR027"
 			(at 187.96 59.69 0)
 			(effects
@@
 			(project "rpi_pico_media_board"
 				(path "/883c739e-d2a5-4bc8-a050-29a6043b4072/373bacf3-831c-41f0-9f95-7ac0a975261a"
-					(reference "#PWR27")
+					(reference "#PWR027")
 					(unit 1)
 				)
@@
 		(in_bom yes)
 		(on_board yes)
-		(dnp no)
+		(dnp yes)
 		(fields_autoplaced yes)
 		(property "Reference" "J301"
@@
 		(dnp no)
 		(fields_autoplaced yes)
-		(property "Reference" "#PWR23"
+		(property "Reference" "#PWR023"
 			(at 156.21 149.86 0)
 			(effects
@@
 			(project "rpi_pico_media_board"
 				(path "/883c739e-d2a5-4bc8-a050-29a6043b4072/373bacf3-831c-41f0-9f95-7ac0a975261a"
-					(reference "#PWR23")
+					(reference "#PWR023")
 					(unit 1)
 				)
@@
 		(dnp no)
 		(fields_autoplaced yes)
-		(property "Reference" "#PWR21"
+		(property "Reference" "#PWR021"
 			(at 134.62 97.79 0)
 			(effects
@@
 			(project "rpi_pico_media_board"
 				(path "/883c739e-d2a5-4bc8-a050-29a6043b4072/373bacf3-831c-41f0-9f95-7ac0a975261a"
-					(reference "#PWR21")
+					(reference "#PWR021")
 					(unit 1)
 				)
