File: KiCad/[4]TF_CARD.kicad_sch (KiCad schematic)
At the start: 14 parts, among them J400 TF-01A

Commit message: Manufacture files preparation
Parts:
- C401: Manufacturer Part Number CL10B104KB8NNNC -> CL10B104KA8NNNC
Changed lines of the file:
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@@
 		(dnp no)
 		(fields_autoplaced yes)
-		(property "Reference" "#PWR37"
+		(property "Reference" "#PWR037"
 			(at 167.64 68.58 0)
 			(effects
@@
 			(project "rpi_pico_media_board"
 				(path "/883c739e-d2a5-4bc8-a050-29a6043b4072/900388d4-7c2a-4794-9944-89b7c592f5cc"
-					(reference "#PWR37")
+					(reference "#PWR037")
 					(unit 1)
 				)
@@
 		(dnp no)
 		(fields_autoplaced yes)
-		(property "Reference" "#PWR38"
+		(property "Reference" "#PWR038"
 			(at 179.07 113.03 0)
 			(effects
@@
 			(project "rpi_pico_media_board"
 				(path "/883c739e-d2a5-4bc8-a050-29a6043b4072/900388d4-7c2a-4794-9944-89b7c592f5cc"
-					(reference "#PWR38")
+					(reference "#PWR038")
 					(unit 1)
 				)
@@
 		(dnp no)
 		(fields_autoplaced yes)
-		(property "Reference" "#PWR36"
+		(property "Reference" "#PWR036"
 			(at 154.94 50.8 0)
 			(effects
@@
 			(project "rpi_pico_media_board"
 				(path "/883c739e-d2a5-4bc8-a050-29a6043b4072/900388d4-7c2a-4794-9944-89b7c592f5cc"
-					(reference "#PWR36")
+					(reference "#PWR036")
 					(unit 1)
 				)
@@
 		(dnp no)
 		(fields_autoplaced yes)
-		(property "Reference" "#PWR39"
+		(property "Reference" "#PWR039"
 			(at 195.58 99.06 0)
 			(effects
@@
 			(project "rpi_pico_media_board"
 				(path "/883c739e-d2a5-4bc8-a050-29a6043b4072/900388d4-7c2a-4794-9944-89b7c592f5cc"
-					(reference "#PWR39")
+					(reference "#PWR039")
 					(unit 1)
 				)
@@
 			)
 		)
-		(property "Manufacturer Part Number" "CL10B104KB8NNNC"
+		(property "Manufacturer Part Number" "CL10B104KA8NNNC"
 			(at 167.64 54.61 0)
 			(effects
@@
 			)
 		)
-		(property "Manufacturer_Name" ""
-			(at 189.23 569.85 0)
-			(effects
-				(font
-					(size 1.27 1.27)
-				)
-				(justify left top)
-				(hide yes)
-			)
-		)
-		(property "Manufacturer_Part_Number" ""
-			(at 189.23 669.85 0)
-			(effects
-				(font
-					(size 1.27 1.27)
-				)
-				(justify left top)
-				(hide yes)
-			)
-		)
-		(property "Mouser Part Number" ""
-			(at 189.23 769.85 0)
-			(effects
-				(font
-					(size 1.27 1.27)
-				)
-				(justify left top)
-				(hide yes)
-			)
-		)
-		(property "Mouser Price/Stock" ""
-			(at 189.23 869.85 0)
-			(effects
-				(font
-					(size 1.27 1.27)
-				)
-				(justify left top)
-				(hide yes)
-			)
-		)
 		(property "Arrow Part Number" ""
 			(at 189.23 969.85 0)
@@
 		(dnp no)
 		(fields_autoplaced yes)
-		(property "Reference" "#PWR34"
+		(property "Reference" "#PWR034"
 			(at 101.6 68.58 0)
 			(effects
@@
 			(project "rpi_pico_media_board"
 				(path "/883c739e-d2a5-4bc8-a050-29a6043b4072/900388d4-7c2a-4794-9944-89b7c592f5cc"
-					(reference "#PWR34")
+					(reference "#PWR034")
 					(unit 1)
 				)
@@
 		(dnp no)
 		(fields_autoplaced yes)
-		(property "Reference" "#PWR35"
+		(property "Reference" "#PWR035"
 			(at 101.6 119.38 0)
 			(effects
@@
 			(project "rpi_pico_media_board"
 				(path "/883c739e-d2a5-4bc8-a050-29a6043b4072/900388d4-7c2a-4794-9944-89b7c592f5cc"
-					(reference "#PWR35")
+					(reference "#PWR035")
 					(unit 1)
 				)
