File: KiCad/[5]Macro_Pad.kicad_sch (KiCad schematic)
At the start: 46 parts, among them Q500 T2N7002AK, Q501 T2N7002AK, Q502 T2N7002AK, U500 SW, U501 SW, U502 SW, U503 SW, U504 SW, U505 SW, U506 SW, U507 SW, U508 SW, U509 SW, U510 SW, U511 SW

Commit message: Manufacture files preparation
Parts:
- C500, C501, C502: Manufacturer Part Number CL10B104KB8NNNC -> CL10B104KA8NNNC
- U500, U501, U502, U503, U504, U505, U506, U507, U508, U509, U510, U511: Manufacturer (none) -> SM Switch; Manufacturer Part Number (none) -> SMG-01-H080A1
