File: KiCad/rpi_pico_media_board.kicad_pcb (KiCad board)
At the start: 4 copper layers, 100 x 80 mm, 138 parts, among them J100 Barrel_Jack_Switch_Pin3Ring, J200 Conn_01x04_Pin, J201 Conn_01x04_Pin, J300 AudioJack3_Ground_SwitchTR, J301 Conn_01x03_Pin, J400 TF-01A, Q100 T2N7002AK, Q500 T2N7002AK, Q501 T2N7002AK, Q502 T2N7002AK, SW200 SW_DPDT_XLX, U100 HT7533-1, U101 HT7533-1, U200 RaspberryPi_Pico, U202 mems-mic, U203 mems-mic, U300 PCM5102A, U500 SW, U501 SW, U502 SW, U503 SW, U504 SW, U505 SW, U506 SW, U507 SW, U508 SW, U509 SW, U510 SW, U511 SW, U600 PCF8563TS, Y600 32768Hz

Commit message: Manufacture files preparation
Other:
- rule pad_to_mask_clearance: 0.038 -> 0

Commit message: Manufacture files
Parts:
- moved D100 0.25 mm to (109.2, 77.8)
- moved D200 0.25 mm to (109.2, 75.5)
- moved D201 0.25 mm to (72.5, 59.5)
- moved D202 0.25 mm to (72.5, 57.0)
- moved D203 0.25 mm to (72.5, 54.5)
- moved SW200 0.21 mm to (105.2, 70.0)
Routing:
- net GND: track 63.3 -> 63.9 mm
